Commit message: Update noetic

File: scout_description/urdf/scout.urdf.xacro (robot description, xacro)
@@ -31,14 +31,14 @@
     <origin xyz="0 0 0.2365" rpy="0 0 0"/>
   </joint>
-  <xacro:scout_wheel prefix="front_left" type="wheel_1">
+  <xacro:scout_wheel prefix="front_left" type="wheel_1" position="left">
     <origin xyz="0.249 0.2915 0.165" rpy="0 0 0"/>
   </xacro:scout_wheel>
-  <xacro:scout_wheel prefix="rear_left" type="wheel_2">
+  <xacro:scout_wheel prefix="rear_left" type="wheel_2" position="left">
     <origin xyz="-0.249 0.2915 0.165" rpy="0 0 0"/>
   </xacro:scout_wheel>
-  <xacro:scout_wheel prefix="front_right" type="wheel_2">
+  <xacro:scout_wheel prefix="front_right" type="wheel_2" position="right">
     <origin xyz="0.249 -0.2915 0.165" rpy="0 0 0"/>
   </xacro:scout_wheel>
-  <xacro:scout_wheel prefix="rear_right" type="wheel_1">
+  <xacro:scout_wheel prefix="rear_right" type="wheel_1" position="right">
     <origin xyz="-0.249 -0.2915 0.165" rpy="0 0 0"/>
   </xacro:scout_wheel>

File: scout_description/urdf/scout_wheel.urdf.xacro (robot description, xacro)
@@ -1,8 +1,13 @@
 <?xml version="1.0"?>
 <robot xmlns:xacro="http://ros.org/wiki/xacro" name="scout_wheel">
-  <xacro:macro name="scout_wheel" params="prefix type *origin">
+  <xacro:macro name="scout_wheel" params="prefix type position *origin">
     <link name="${prefix}_wheel">
       <visual>
-        <origin xyz="0.0 0.0 0.0" rpy="0 0 0"/>
+        <xacro:if value="${position == 'left'}">
+          <origin xyz="0.0 0.0 0.0" rpy="0 0 0"/>
+        </xacro:if>
+        <xacro:if value="${position == 'right'}">
+          <origin xyz="0.0 0.0 0.0" rpy="${PI} 0 0"/>
+        </xacro:if>
         <geometry>
           <mesh filename="package://scout_description/meshes/${type}.dae"/>

Commit message: 0.2.2

File: scout_description/urdf/scout.urdf.xacro (robot description, xacro)
@@ -1,17 +1,17 @@
 <?xml version="1.0"?>
 <robot xmlns:xacro="http://www.ros.org/wiki/xacro" name="scout">
-  <xacro:include filename="$(find scout_description)/urdf/scout_wheel.urdf.xacro"/>
-  <xacro:property name="PI" value="3.1415926535897931"/>
+  <xacro:include filename="$(find scout_description)/urdf/scout_wheel.urdf.xacro" />
+  <xacro:property name="PI" value="3.1415926535897931" />
   <link name="base_link">
     <visual>
-      <origin xyz="0.0 0.0 0.2365" rpy="0 0 0"/>
+      <origin xyz="0.0 0.0 0.2365" rpy="0 0 0" />
       <geometry>
-        <mesh filename="package://scout_description/meshes/scout.dae"/>
+        <mesh filename="package://scout_description/meshes/scout.dae" />
       </geometry>
     </visual>
     <collision>
-      <origin xyz="0.0 0.0 0.2365" rpy="0 0 0"/>
+      <origin xyz="0.0 0.0 0.2365" rpy="0 0 0" />
       <geometry>
-        <mesh filename="package://scout_description/meshes/scout.dae"/>
+        <mesh filename="package://scout_description/meshes/scout.dae" />
       </geometry>
     </collision>
@@ -19,27 +19,27 @@
   <link name="inertial_link">
     <inertial>
-      <mass value="40"/>
-      <origin rpy=" 0 0 0" xyz="0 0 0"/>
+      <mass value="40" />
+      <origin rpy=" 0 0 0" xyz="0 0 0" />
       <!--inertia ixx="2.288641" ixy="0.0" ixz="0.0" iyy="5.103976" iyz="0.0" izz="3.431465"/-->
-      <inertia ixx="2.42811" ixy="0.00503" ixz="0.09703" iyy="2.52291" iyz="0.10757" izz="0.18274"/>
+      <inertia ixx="2.42811" ixy="0.00503" ixz="0.09703" iyy="2.52291" iyz="0.10757" izz="0.18274" />
       <!--inertia ixx="0.6022" ixy="-0.02364" ixz="-0.1197" iyy="1.7386" iyz="-0.001544" izz="2.0296"/-->
     </inertial>
   </link>
   <joint name="inertial_joint" type="fixed">
-    <parent link="base_link"/>
-    <child link="inertial_link"/>
-    <origin xyz="0 0 0.2365" rpy="0 0 0"/>
+    <parent link="base_link" />
+    <child link="inertial_link" />
+    <origin xyz="0 0 0.2365" rpy="0 0 0" />
   </joint>
   <xacro:scout_wheel prefix="front_left" type="wheel_1" position="left">
-    <origin xyz="0.249 0.2915 0.165" rpy="0 0 0"/>
+    <origin xyz="0.249 0.2915 0.165" rpy="0 0 0" />
   </xacro:scout_wheel>
   <xacro:scout_wheel prefix="rear_left" type="wheel_2" position="left">
-    <origin xyz="-0.249 0.2915 0.165" rpy="0 0 0"/>
+    <origin xyz="-0.249 0.2915 0.165" rpy="0 0 0" />
   </xacro:scout_wheel>
   <xacro:scout_wheel prefix="front_right" type="wheel_2" position="right">
-    <origin xyz="0.249 -0.2915 0.165" rpy="0 0 0"/>
+    <origin xyz="0.249 -0.2915 0.165" rpy="0 0 0" />
   </xacro:scout_wheel>
   <xacro:scout_wheel prefix="rear_right" type="wheel_1" position="right">
-    <origin xyz="-0.249 -0.2915 0.165" rpy="0 0 0"/>
+    <origin xyz="-0.249 -0.2915 0.165" rpy="0 0 0" />
   </xacro:scout_wheel>
   <gazebo>

File: scout_description/urdf/scout_wheel.urdf.xacro (robot description, xacro)
@@ -5,41 +5,41 @@
       <visual>
         <xacro:if value="${position == 'left'}">
-          <origin xyz="0.0 0.0 0.0" rpy="0 0 0"/>
+          <origin xyz="0.0 0.0 0.0" rpy="0 0 0" />
         </xacro:if>
         <xacro:if value="${position == 'right'}">
-          <origin xyz="0.0 0.0 0.0" rpy="${PI} 0 0"/>
+          <origin xyz="0.0 0.0 0.0" rpy="${PI} 0 0" />
         </xacro:if>
         <geometry>
-          <mesh filename="package://scout_description/meshes/${type}.dae"/>
+          <mesh filename="package://scout_description/meshes/${type}.dae" />
         </geometry>
       </visual>
       <collision>
-        <origin xyz="0.0 0.0 0.0" rpy="0 0 0"/>
+        <origin xyz="0.0 0.0 0.0" rpy="0 0 0" />
         <geometry>
-          <mesh filename="package://scout_description/meshes/${type}.dae"/>
+          <mesh filename="package://scout_description/meshes/${type}.dae" />
         </geometry>
       </collision>
       <inertial>
-        <mass value="3"/>
-        <origin xyz="0.0 0.0 0.0" rpy="0 0 0"/>
+        <mass value="3" />
+        <origin xyz="0.0 0.0 0.0" rpy="0 0 0" />
         <!--inertia ixx="0.7171" ixy="0.0" ixz="0.0" iyy="0.1361" iyz="0.0" izz="0.7171"/-->
-        <inertia ixx="0.02467" ixy="0" ixz="0" iyy="0.04411" iyz="0" izz="0.02467"/>
+        <inertia ixx="0.02467" ixy="0" ixz="0" iyy="0.04411" iyz="0" izz="0.02467" />
       </inertial>
     </link>
     <joint name="${prefix}_wheel_joint" type="continuous">
-      <parent link="base_link"/>
-      <child link="${prefix}_wheel"/>
-      <xacro:insert_block name="origin"/>
-      <axis xyz="0 1 0" rpy="0 0 0"/>
+      <parent link="base_link" />
+      <child link="${prefix}_wheel" />
+      <xacro:insert_block name="origin" />
+      <axis xyz="0 1 0" rpy="0 0 0" />
       <!--limit effort="200" velocity="200"/>
       <joint_properties damping="0" friction="0"/-->
     </joint>
     <gazebo reference="${prefix}_wheel">
-      <mu1 value="1.0"/>
-      <mu2 value="1.0"/>
-      <fdir1 value="1 0 0"/>
-      <kp value="10000000.0"/>
-      <kd value="1.0"/>
-      <minDepth value="0.001"/>
+      <mu1 value="1.0" />
+      <mu2 value="1.0" />
+      <fdir1 value="1 0 0" />
+      <kp value="10000000.0" />
+      <kd value="1.0" />
+      <minDepth value="0.001" />
       <!--turnGravityOff>false</turnGravityOff-->
     </gazebo>
